File: _autosave-male_keyboard.kicad_pcb (KiCad board)
At the start: 2 copper layers, 1 part, among them J1 Elite-Pi Microcontroller

Commit message: 15042025
Parts:
- added J2: AudioJack4, Keebio-Parts:TRRS-PJ-320A, F.Cu at (34.8, 87.3)
- added SW1: SW_MEC_5G, Button_Switch_Keyboard:SW_Cherry_MX_1.00u_PCB, F.Cu at (101.5, 22.4)
- moved J1 36.6 mm to (64.5, 56.8)
Connections:
- J1 pad 19: unconnected-(J1-Pin_19-Pad19) -> Net-(J1-Pin_19)
- J1 pad 2: unconnected-(J1-Pin_2-Pad2) -> Net-(J1-Pin_2)
- J1 pad 21: unconnected-(J1-Pin_21-Pad21) -> Net-(J1-Pin_21)
- J1 pad 23: unconnected-(J1-Pin_23-Pad23) -> GND
