File: male_keyboard.kicad_pcb (KiCad board)
At the start: 2 copper layers, 0 parts

Commit message: 15042025
Parts:
- added J1: Elite-Pi Microcontroller, Keebio-Parts:Elite-C, F.Cu at (33.5, 37.3)
