File: male_keyboard.kicad_pcb (KiCad board)
At the start: 2 copper layers, 40 parts, among them J1 Elite-Pi Microcontroller, J2 AudioJack4, J3 AudioJack4, J4 Elite-Pi Microcontroller, SW1 SW_Push, SW10 SW_Push, SW11 SW_Push, SW12 SW_Push, SW13 SW_Push, SW14 SW_Push, SW15 SW_Push, SW16 SW_Push, SW17 SW_Push, SW18 SW_Push, SW19 SW_Push, SW2 SW_Push, SW20 SW_Push, SW21 SW_Push, SW22 SW_Push, SW23 SW_Push, SW24 SW_Push, SW25 SW_Push, SW26 SW_Push, SW27 SW_Push, SW28 SW_Push, SW29 SW_Push, SW3 SW_Push, SW30 SW_Push, SW31 SW_Push, SW32 SW_Push, SW33 SW_Push, SW34 SW_Push, SW35 SW_Push, SW36 SW_Push, SW4 SW_Push, SW5 SW_Push, SW6 SW_Push, SW7 SW_Push, SW8 SW_Push, SW9 SW_Push

Commit message: positioning right
Parts:
- moved SW18 19.3 mm to (116.5, 121.4)
- moved SW17 16.2 mm to (95.8, 117.5)
- moved SW16 14.1 mm to (76.5, 117.4)
- moved SW32 12.4 mm to (232.0, 90.0)
- moved SW27 10.5 mm to (232.0, 70.0)
- moved SW15 10.1 mm to (104.5, 98.0)
- moved SW14 8.93 mm to (85.5, 98.0)
- moved SW13 8.50 mm to (66.5, 98.0)
- moved SW21 8.23 mm to (232.0, 50.0)
- moved SW12 7.76 mm to (47.5, 98.0)
- moved SW5 7.44 mm to (104.6, 60.0)
- moved SW10 7.23 mm to (104.5, 78.9)
- moved SW11 7.05 mm to (28.5, 98.0)
- moved SW4 6.12 mm to (85.5, 59.9)
- moved SW9 5.67 mm to (85.5, 78.9)
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Routing:
- net 1: track 96.9 -> 1.01 mm
- net 2: track 76.1 -> 0.00 mm
- net GND: track 65.5 -> 2.05 mm
- net 3: track 57.6 -> 0.00 mm
- net 4: track 38.5 -> 3.51 mm

Commit message: finish locking
Parts:
- moved SW34 113.1 mm to (169.5, 144.5), turned to 45 degrees
- moved SW33 98.2 mm to (272.0, 110.0)
- moved SW29 84.8 mm to (192.0, 100.0)
- moved SW24 82.4 mm to (192.0, 80.0)
- moved SW18 39.1 mm to (145.0, 148.2), turned to -45 degrees
- moved SW35 35.6 mm to (188.5, 129.5), turned to 30 degrees
- moved SW17 34.5 mm to (126.7, 132.9), turned to -30 degrees
- moved SW16 28.9 mm to (104.9, 122.9), turned to -15 degrees
- moved SW23 21.9 mm to (272.0, 70.0)
- moved SW27 21.9 mm to (252.0, 79.0)
- moved SW28 21.9 mm to (272.0, 90.0)
- moved SW32 21.9 mm to (252.0, 99.0)
- moved SW26 21.2 mm to (232.0, 70.0)
- moved SW31 21.2 mm to (232.0, 90.0)
- moved SW25 20.2 mm to (212.0, 77.0)
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Routing:
- net 4: track 3.51 -> 0.00 mm
- net 9: track 0.00 -> 1.24 mm
- net 15: track 1.24 -> 0.00 mm
- net 1: track 1.01 -> 0.00 mm
