File: male_keyboard.kicad_pcb (KiCad board)
At the start: 2 copper layers, 249.7 x 119.1 mm, 40 parts, among them J1L1 Elite-Pi Microcontroller, J2L1 AudioJackLeft, J3R1 Elite-Pi Microcontroller, J4R1 AudioJackRight, SW1 SW_Push, SW10 SW_Push, SW11 SW_Push, SW12 SW_Push, SW13 SW_Push, SW14 SW_Push, SW15 SW_Push, SW16 SW_Push, SW17 SW_Push, SW18 SW_Push, SW19 SW_Push, SW2 SW_Push, SW20 SW_Push, SW21 SW_Push, SW22 SW_Push, SW23 SW_Push, SW24 SW_Push, SW25 SW_Push, SW26 SW_Push, SW27 SW_Push, SW28 SW_Push, SW29 SW_Push, SW3 SW_Push, SW30 SW_Push, SW31 SW_Push, SW32 SW_Push, SW33 SW_Push, SW34 SW_Push, SW35 SW_Push, SW36 SW_Push, SW4 SW_Push, SW5 SW_Push, SW6 SW_Push, SW7 SW_Push, SW8 SW_Push, SW9 SW_Push

Commit message: rounded edges
Other:
- board size 249.7 x 119.1 mm -> 249.7 x 118.9 mm
